File: eagle/pt2399_echo.brd (EAGLE design)
At the start: 100 x 80 mm, 35 parts

Commit message: corrected, rerouted, gcode
Parts:
- removed POT: 50k, pot:3RP/1610N
- added FEEDBACK: 50k, pot:3RP/1610N
- C13, C22: device rcl:C025-024X044 -> rcl:C050-024X044
- C17, C18, C25, C26: device rcl:C050-025X075 -> rcl:C050-024X044
- R1, R10, R2, R3, R4, R5, R6, R7, R8, R9: device rcl:0207/10 -> rcl:0207/7
- R11: value 10k -> 1k
- TIME: value 20k -> 50k
- moved IN_LEVEL 83.8 mm to (3.81, 58.4), turned to 270 degrees
- moved OUT 81.7 mm to (0.00, 68.6), turned to 90 degrees
- moved R7 73.6 mm to (12.4, 27.2), turned to 0 degrees
- moved R1 71.4 mm to (11.4, 61.0), turned to 270 degrees
- moved INPUT 68.8 mm to (0.00, 38.4), turned to 90 degrees
- moved C24 67.6 mm to (12.2, 23.1), turned to 270 degrees
- moved C16 67.5 mm to (16.5, 55.9), turned to 180 degrees
- moved C19 60.2 mm to (16.3, 31.0), turned to 180 degrees
- moved R2 55.1 mm to (22.9, 52.1), turned to 270 degrees
- moved C23 51.5 mm to (20.1, 63.8)
- moved C11 46.0 mm to (23.1, 17.3), turned to 270 degrees
- moved C17 45.6 mm to (27.2, 48.3), turned to 0 degrees
- moved R3 42.6 mm to (22.9, 40.6), turned to 270 degrees
- moved C15 40.3 mm to (17.8, 12.7), turned to 0 degrees
- moved C18 38.1 mm to (22.9, 34.3), turned to 0 degrees
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Connections:
- removed net GND: IC2.4, PWR1.3, PWR1.4, PWR1.5, PWR1.6, PWR1.7, PWR1.8, TIME.1, TIME.2
- net AGND: now also FEEDBACK.1, IC2.4, PWR1.3, PWR1.4, PWR1.5, PWR1.6, PWR1.7, PWR1.8, TIME.1; no longer POT.3
- net N$20: now also FEEDBACK.2; no longer POT.2
- net N$22: now also FEEDBACK.3; no longer POT.1
- net N$28: now also TIME.2
Routing:
- net N$21: track 161.7 -> 42.4 mm
- net GND: track 114.1 -> 0.00 mm
- net AGND: track 171.8 -> 253.9 mm
- net N$29: track 39.4 -> 9.93 mm
- net +5V: track 39.8 -> 16.8 mm
- net N$28: track 7.64 -> 27.4 mm
- net N$7: track 0.00 -> 17.8 mm
- net N$11: track 10.1 -> 25.0 mm
- net N$17: track 0.00 -> 10.4 mm
- net N$14: track 11.7 -> 3.05 mm
- net N$5: track 9.67 -> 2.74 mm
- net N$19: track 10.7 -> 4.11 mm
- net N$9: track 11.2 -> 5.08 mm
- net N$25: track 13.9 -> 7.98 mm
- net N$4: track 8.60 -> 3.87 mm
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Other:
- board size 100 x 80 mm -> 100.8 x 80.5 mm
