File: eagle/pt2399_echo.sch (EAGLE design)
At the start: 35 parts

Commit message: corrected, rerouted, gcode
Parts:
- C13, C22: device rcl:C-US025-024X044 -> rcl:C-US050-024X044
- C17, C18, C25, C26: device rcl:C-US050-025X075 -> rcl:C-US050-024X044
- R1, R10, R2, R3, R4, R5, R6, R7, R8, R9: device rcl:R-US_0207/10 -> rcl:R-US_0207/7
- R11: value 10k -> 1k
- TIME: value 20k -> 50k
- renumbered POT to FEEDBACK
Connections:
- removed net GND: IC2.DGND, PWR1.GND, TIME.A, TIME.S
- net AGND: now also FEEDBACK.A, IC2.DGND, PWR1.GND, TIME.A; no longer FEEDBACK.E
- net N$22: now also FEEDBACK.E; no longer FEEDBACK.A
- net N$28: now also TIME.S
Other:
- moved on the sheet: TIME
